File: pcb/pcb.kicad_pcb (KiCad board)
At the start: 2 copper layers, 100 x 31 mm, 24 parts, among them J1 USB_C_Receptacle_USB2.0_16P, J2 USB_A, J3 USB_A, J4 USB_A, J5 USB_A, U1 SL2.1A

Commit message: Update PCB
Other:
- board size 100 x 31 mm -> 99 x 31 mm
Changed lines of the file:
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@@
 	(gr_rect
 		(start 87.357 69.172)
-		(end 187.357 100.172)
+		(end 186.357 100.172)
 		(stroke
 			(width 0.05)
@@
 		(polygon
 			(pts
-				(xy 87.25 69) (xy 187.75 69) (xy 187.75 100.25) (xy 87.25 100.25)
+				(xy 87.25 69) (xy 186.45 69) (xy 186.45 100.25) (xy 87.25 100.25)
 			)
 		)
